Commit message: solved small issue with collision meshes

File: mobile_manipulator_ws/src/robot_description/urdf/robot_base.urdf.xacro (robot description, xacro)
@@ -1,22 +1,21 @@
 <?xml version="1.0"?>
-<robot xmlns:xacro="http://www.ros.org/wiki/xacro" name="robot_base">
+<robot xmlns:xacro="http://ros.org/wiki/xacro" name="robot_base">
     <xacro:include filename="$(find robot_description)/urdf/robot_base_essentials.xacro" />
     <xacro:include filename="$(find robot_description)/urdf/gazebo_base_essentials.xacro" />
     <!--############################# Base Link #########################################-->
-    <link name="world"/>
     <link name="base_link">
         <inertial>
             <origin
-                xyz="-4.1867E-18 0.0068085 -1.65658661799998E-18"
+                xyz="0.0030946 4.78250032638821E-11 0.053305"
                 rpy="0 0 0" />
             <mass
-                value="2.6578" />
+                value="47.873" />
             <inertia
-                ixx="0.00856502765719703"
-                ixy="1.5074118157338E-19"
-                ixz="-4.78150098725052E-19"
-                iyy="0.013670640432096"
-                iyz="-2.68136447099727E-19"
-                izz="0.00856502765719703" />
+                ixx="0.774276574699151"
+                ixy="-1.03781944357671E-10"
+                ixz="0.00763014265820928"
+                iyy="1.64933255189991"
+                iyz="1.09578155845563E-12"
+                izz="2.1239326987473" />
         </inertial>
         <visual>
@@ -42,9 +41,4 @@
         </collision>
     </link>
-    <joint name="virtual_joint" type="fixed">
-        <parent link="world"/>
-        <child link="base_link"/>
-        <origin xyz="0 0 0"/>
-    </joint>
     <!--############################# Wheel Links #########################################-->
     <xacro:robot_wheel prefix="front_left"/>

File: mobile_manipulator_ws/src/robot_description/urdf/robot_base_essentials.xacro (robot description, xacro)
@@ -1,19 +1,19 @@
 <?xml version="1.0"?>
-<robot xmlns:xacro="http://www.ros.org/wiki/xacro">
+<robot xmlns:xacro="http://ros.org/wiki/xacro" name="robot_base_essentials">
     <xacro:macro name="robot_wheel" params="prefix">
         <link name="${prefix}_wheel">
             <inertial>
                 <origin
-                    xyz="0.0030946 4.78250032638821E-11 0.053305"
+                    xyz="-4.1867E-18 0.0068085 -1.65658661799998E-18"
                     rpy="0 0 0" />
                 <mass
-                    value="47.873" />
+                    value="2.6578" />
                 <inertia
-                    ixx="0.774276574699151"
-                    ixy="-1.03781944357671E-10"
-                    ixz="0.00763014265820928"
-                    iyy="1.64933255189991"
-                    iyz="1.09578155845563E-12"
-                    izz="2.1239326987473" />
+                    ixx="0.00856502765719703"
+                    ixy="1.5074118157338E-19"
+                    ixz="-4.78150098725052E-19"
+                    iyy="0.013670640432096"
+                    iyz="-2.68136447099727E-19"
+                    izz="0.00856502765719703" />
             </inertial>
             <visual>
@@ -35,5 +35,5 @@
                     rpy="1.5707963267949 0 0" />
                 <geometry>
-                    <mesh filename="package://robot_description/meshes/robot_base.stl" />
+                    <mesh filename="package://robot_description/meshes/wheel.stl" />
                 </geometry>
             </collision>
