Commit message: added urdf model for the complete robot

File: mobile_manipulator_ws/src/robot_description/urdf/gazebo_arm_essentials.xacro (robot description, xacro)
@@ -1,17 +1,21 @@
 <?xml version="1.0"?>
 <robot xmlns:xacro="http://www.ros.org/wiki/xacro" name="gazebo_arm_essentials">
-<!--############################# ROS-CONTROL #########################################-->
+  <!--############################# ROS-CONTROL #########################################-->
+  <xacro:macro name="gazebo_ros_control">
     <gazebo>
-        <plugin name="gazebo_ros_control" filename="libgazebo_ros_control.so">
-            <robotNamespace>/</robotNamespace>
-            <controlPeriod>0.001</controlPeriod>
-            <legacyModeNS>false</legacyModeNS>
-        </plugin>
+      <plugin name="gazebo_ros_control" filename="libgazebo_ros_control.so">
+        <robotNamespace>/</robotNamespace>
+        <controlPeriod>0.001</controlPeriod>
+        <legacyModeNS>false</legacyModeNS>
+      </plugin>
     </gazebo>
-<!--################################ ROS-Controllers ######################################-->
-  <gazebo>
-    <plugin name="joint_state_publisher" filename="libgazebo_ros_joint_state_publisher.so">
-      <jointName>arm_base_joint, shoulder_joint, bottom_wrist_joint, elbow_joint, bottom_wrist_joint</jointName>
-    </plugin>
-  </gazebo>
+  </xacro:macro>
+  <!--################################ ROS-Controllers ######################################-->
+  <xacro:macro name="joint_state_publisher">
+    <gazebo>
+      <plugin name="joint_state_publisher" filename="libgazebo_ros_joint_state_publisher.so">
+        <jointName>arm_base_joint, shoulder_joint, bottom_wrist_joint, elbow_joint, bottom_wrist_joint</jointName>
+      </plugin>
+    </gazebo>
+  </xacro:macro>
 </robot>

File: mobile_manipulator_ws/src/robot_description/urdf/gazebo_base_essentials.xacro (robot description, xacro)
@@ -1,44 +1,48 @@
 <?xml version="1.0"?>
 <robot xmlns:xacro="http://www.ros.org/wiki/xacro" name="gazebo_base_essentials">
-<!--############################# ROS-CONTROL #########################################-->
-    <gazebo>
-        <plugin name="gazebo_ros_control" filename="libgazebo_ros_control.so">
-        <robotNamespace>/</robotNamespace>
-        <controlPeriod>0.001</controlPeriod>
-        <legacyModeNS>false</legacyModeNS>
-        </plugin>
-    </gazebo>
-<!--################################ ROS-Controllers ######################################-->
-    <gazebo>
-        <plugin name="diff_drive_controller" filename="libgazebo_ros_diff_drive.so">
-            <legacyMode>false</legacyMode>
-            <alwaysOn>true</alwaysOn>
-            <updateRate>1000.0</updateRate>
-            <leftJoint>front_left_wheel_joint, rear_left_wheel_joint</leftJoint>
-            <rightJoint>front_right_wheel_joint, rear_right_wheel_joint</rightJoint>
-            <wheelSeparation>0.5</wheelSeparation>
-            <wheelDiameter>0.2</wheelDiameter>
-            <wheelTorque>10</wheelTorque>
-            <publishTf>1</publishTf>
-            <odometryFrame>map</odometryFrame>
-            <commandTopic>cmd_vel</commandTopic>
-            <odometryTopic>odom</odometryTopic>
-            <robotBaseFrame>base_link</robotBaseFrame>
-            <wheelAcceleration>2.8</wheelAcceleration>
-            <publishWheelJointState>true</publishWheelJointState>
-            <publishWheelTF>false</publishWheelTF>
-            <odometrySource>world</odometrySource>
-            <rosDebugLevel>Debug</rosDebugLevel>
-        </plugin>
-    </gazebo>
-<!--############################# Wheel friction #########################################-->
-<xacro:macro name="wheel_friction" params="prefix ">
-    <gazebo reference="${prefix}_wheel">
-        <mu1 value="1.0"/>
-        <mu2 value="1.0"/>
-        <kp value="10000000.0" />
-        <kd value="1.0" />
-        <fdir1 value="1 0 0"/>
-    </gazebo>
-</xacro:macro>
+    <!--############################# ROS-CONTROL #########################################-->
+    <xacro:macro name="gazebo_ros_control">
+        <gazebo>
+            <plugin name="gazebo_ros_control" filename="libgazebo_ros_control.so">
+                <robotNamespace>/</robotNamespace>
+                <controlPeriod>0.001</controlPeriod>
+                <legacyModeNS>false</legacyModeNS>
+            </plugin>
+        </gazebo>
+    </xacro:macro>
+    <!--################################ ROS-Controllers ######################################-->
+    <xacro:macro name="diff_drive_controller">
+        <gazebo>
+            <plugin name="diff_drive_controller" filename="libgazebo_ros_diff_drive.so">
+                <legacyMode>false</legacyMode>
+                <alwaysOn>true</alwaysOn>
+                <updateRate>1000.0</updateRate>
+                <leftJoint>front_left_wheel_joint, rear_left_wheel_joint</leftJoint>
+                <rightJoint>front_right_wheel_joint, rear_right_wheel_joint</rightJoint>
+                <wheelSeparation>0.5</wheelSeparation>
+                <wheelDiameter>0.2</wheelDiameter>
+                <wheelTorque>10</wheelTorque>
+                <publishTf>1</publishTf>
+                <odometryFrame>map</odometryFrame>
+                <commandTopic>cmd_vel</commandTopic>
+                <odometryTopic>odom</odometryTopic>
+                <robotBaseFrame>base_link</robotBaseFrame>
+                <wheelAcceleration>2.8</wheelAcceleration>
+                <publishWheelJointState>true</publishWheelJointState>
+                <publishWheelTF>false</publishWheelTF>
+                <odometrySource>world</odometrySource>
+                <rosDebugLevel>Debug</rosDebugLevel>
+            </plugin>
+        </gazebo>
+    </xacro:macro>
+    <!--############################# Wheel friction #########################################-->
+    <xacro:macro name="wheel_friction" params="prefix ">
+        <gazebo reference="${prefix}_wheel">
+            <mu1 value="1.0"/>
+            <mu2 value="1.0"/>
+            <kp value="10000000.0" />
+            <kd value="1.0" />
+            <fdir1 value="1 0 0"/>
+        </gazebo>
+    </xacro:macro>
 </robot>

File: mobile_manipulator_ws/src/robot_description/urdf/mobile_manipulator.urdf.xacro (robot description, xacro)
@@ -1,6 +1,68 @@
 <?xml version="1.0"?>
-<robot xmlns:xacro="http://ros.org/wiki/xacro" name="mobile_manipulator" >
-    <xacro:include filename="$(find robot_description)/urdf/robot_base.urdf.xacro" />
-    <xacro:include filename="$(find robot_description)/urdf/robot_arm.urdf.xacro" />
-    <xacro:arm_joint prefix="arm_base_link" type="continuous" axis="0 0 1" parent="base_link" child="arm_base" originxyz="0.20 0.0 0.145" originrpy="0 0 0"/>
+<robot xmlns:xacro="http://ros.org/wiki/xacro" name="mobile_manipulator">
+  <!--################################# BASE LINKS #####################################-->
+  <xacro:include filename="$(find robot_description)/urdf/robot_base_essentials.xacro" />
+  <xacro:include filename="$(find robot_description)/urdf/gazebo_base_essentials.xacro" />
+  <link name="base_link">
+    <inertial>
+      <origin xyz="0.0030946 4.78250032638821E-11 0.053305" rpy="0 0 0" />
+      <mass value="47.873" />
+      <inertia ixx="0.774276574699151" ixy="-1.03781944357671E-10" ixz="0.00763014265820928" iyy="1.64933255189991" iyz="1.09578155845563E-12" izz="2.1239326987473" />
+    </inertial>
+    <visual>
+      <origin xyz="0 0 0" rpy="1.5707963267949 0 3.14" />
+      <geometry>
+        <mesh filename="package://robot_description/meshes/robot_base.stl" />
+      </geometry>
+      <material name="">
+        <color rgba="0.79216 0.81961 0.93333 1" />
+      </material>
+    </visual>
+    <collision>
+      <origin xyz="0 0 0" rpy="1.5707963267949 0 3.14" />
+      <geometry>
+        <mesh filename="package://robot_description/meshes/robot_base.stl" />
+      </geometry>
+    </collision>
+  </link>
+  <xacro:robot_wheel prefix="front_left"/>
+  <xacro:robot_wheel prefix="front_right"/>
+  <xacro:robot_wheel prefix="rear_left"/>
+  <xacro:robot_wheel prefix="rear_right"/>
+  <!--############################## ARM LINKS ########################################-->
+  <xacro:include filename="$(find robot_description)/urdf/robot_arm_essentials.xacro" />
+  <xacro:include filename="$(find robot_description)/urdf/gazebo_arm_essentials.xacro" />
+  <xacro:arm attach="false"/>
+  <!--############################## BASE JOINTS ########################################-->
+  <xacro:wheel_joint prefix="front_left" origin="0.220 0.250 0"/>
+  <xacro:wheel_joint prefix="front_right" origin="0.220 -0.250 0"/>
+  <xacro:wheel_joint prefix="rear_left" origin="-0.220 0.250 0"/>
+  <xacro:wheel_joint prefix="rear_right" origin="-0.220 -0.250 0"/>
+  <!--############################## ARM JOINTS ########################################-->
+  <xacro:arm_joint prefix="arm_world" type="fixed" axis="0 0 1" parent="base_link" child="arm_world" originxyz="0.20 0.0 0.145" originrpy="0 0 0"/>
+  <xacro:arm_joint prefix="arm_base" type="continuous" axis="0 0 1" parent="arm_world" child="arm_base" originxyz="0.0 0.0 0.0" originrpy="0 0 0"/>
+  <xacro:arm_joint prefix="shoulder" type="continuous" axis="0 1 0" parent="arm_base" child="bicep" originxyz="-0.05166 0.0 0.20271" originrpy="0 0 1.5708"/>
+  <xacro:arm_joint prefix="bottom_wrist" type="continuous" axis="0 1 0" parent="bicep" child="bottom_wrist" originxyz="0.0 -0.05194 0.269" originrpy="0 0 0"/>
+  <xacro:arm_joint prefix="elbow" type="continuous" axis="0 0 1" parent="bottom_wrist" child="elbow" originxyz="0.0 0 0.13522" originrpy="0 0 0"/>
+  <xacro:arm_joint prefix="top_wrist" type="continuous" axis="0 1 0" parent="elbow" child="top_wrist" originxyz="0.0 0 0.20994" originrpy="0 0 0"/>
+  <!--############################# BASE TRANSMISSIONS #########################################-->
+  <xacro:base_transmission prefix="front_left"/>
+  <xacro:base_transmission prefix="front_right"/>
+  <xacro:base_transmission prefix="rear_left"/>
+  <xacro:base_transmission prefix="rear_right"/>
+  <!--############################# ARM TRANSMISSION ##################################-->
+  <xacro:arm_transmission prefix="arm_base"/>
+  <xacro:arm_transmission prefix="shoulder"/>
+  <xacro:arm_transmission prefix="bottom_wrist"/>
+  <xacro:arm_transmission prefix="elbow"/>
+  <xacro:arm_transmission prefix="top_wrist"/>
+  <!--############################# WHEEL FRICTIONS #########################################-->
+  <xacro:wheel_friction prefix="front_left"/>
+  <xacro:wheel_friction prefix="front_right"/>
+  <xacro:wheel_friction prefix="rear_left"/>
+  <xacro:wheel_friction prefix="rear_right"/>
+  <!--############################# GAZEBO #########################################-->
+  <xacro:gazebo_ros_control/>
+  <xacro:diff_drive_controller/>
+  <xacro:joint_state_publisher />
 </robot>

File: mobile_manipulator_ws/src/robot_description/urdf/robot_arm.urdf.xacro (robot description, xacro)
@@ -1,204 +1,16 @@
 <?xml version="1.0"?>
-<robot xmlns:xacro="http://ros.org/wiki/xacro" name="robot_arm" >
+<robot xmlns:xacro="http://ros.org/wiki/xacro" name="robot_arm">
     <xacro:include filename="$(find robot_description)/urdf/robot_arm_essentials.xacro" />
     <xacro:include filename="$(find robot_description)/urdf/gazebo_arm_essentials.xacro" />
-    <!--############################# Arm Links #########################################-->
-    <link name="world"/>
-    <link name="arm_base">
-        <inertial>
-            <origin
-                xyz="7.7128E-09 -0.063005 -3.01969999961422E-08"
-                rpy="0 0 0" />
-            <mass
-                value="1.6004" />
-            <inertia
-                ixx="0.00552196561445819"
-                ixy="7.9550614501301E-10"
-                ixz="-1.34378458924839E-09"
-                iyy="0.00352397447953875"
-                iyz="-1.10071809773382E-08"
-                izz="0.00553739792746489" />
-        </inertial>
-        <visual>
-            <origin
-                xyz="0 0 0"
-                rpy="0 0 0" />
-            <geometry>
-                <mesh filename="package://robot_description/meshes/arm_base.stl" />
-            </geometry>
-            <material
-                name="">
-                <color
-                rgba="0.79216 0.81961 0.93333 1" />
-            </material>
-        </visual>
-        <collision>
-            <origin
-                xyz="0 0 0"
-                rpy="0 0 0" />
-            <geometry>
-                <mesh filename="package://robot_description/meshes/arm_base.stl" />
-            </geometry>
-        </collision>
-    </link>
-    <link
-        name="bicep">
-        <inertial>
-            <origin
-                xyz="0.12821 3.5589E-06 0.052492"
-                rpy="0 0 0" />
-            <mass
-                value="1.1198" />
-            <inertia
-                ixx="0.0012474"
-                ixy="-5.4004E-07"
-                ixz="-0.0013148"
-                iyy="0.0072923"
-                iyz="-1.8586E-07"
-                izz="0.0068178" />
-        </inertial>
-        <visual>
-            <origin
-                xyz="0 0 0"
-                rpy="0 -1.5708 0" />
-            <geometry>
-                <mesh filename="package://robot_description/meshes/bicep.stl" />
-            </geometry>
-            <material
-                name="">
-                <color
-                rgba="0.79216 0.81961 0.93333 1" />
-            </material>
-        </visual>
-        <collision>
-            <origin
-                xyz="0 0 0"
-                rpy="0 -1.5708 0" />
-            <geometry>
-                <mesh filename="package://robot_description/meshes/bicep.stl" />
-            </geometry>
-        </collision>
-    </link>
-    <link
-        name="bottom_wrist">
-        <inertial>
-            <origin
-                xyz="-9.1053E-08 -0.069257 -1.86629999995759E-07"
-                rpy="0 0 0" />
-            <mass
-                value="0.27721" />
-            <inertia
-                ixx="0.00104290750143942"
-                ixy="4.37155302268076E-09"
-                ixz="-2.45049603914627E-09"
-                iyy="0.000380518373895034"
-                iyz="-7.56009835172156E-09"
-                izz="0.00106006525067445" />
-        </inertial>
-        <visual>
-            <origin
-                xyz="0 0 0.13522"
-                rpy="3.14 0 1.5708" />
-            <geometry>
-                <mesh filename="package://robot_description/meshes/wrist.stl" />
-            </geometry>
-            <material
-                name="">
-                <color
-                rgba="0.79216 0.81961 0.93333 1" />
-            </material>
-        </visual>
-        <collision>
-            <origin
-                xyz="0 0 0.13522"
-                rpy="3.14 0 1.5708" />
-            <geometry>
-                <mesh filename="package://robot_description/meshes/wrist.stl" />
-            </geometry>
-        </collision>
-    </link>
-    <link
-        name="elbow">
-        <inertial>
-            <origin
-                xyz="-0.11109 1.1476E-08 0.046469"
-                rpy="0 0 0" />
-            <mass
-                value="0.84845" />
-            <inertia
-                ixx="0.00079656"
-                ixy="-7.8011E-10"
-                ixz="0.00053616"
-                iyy="0.003576"
-                iyz="4.6326E-10"
-                izz="0.0033698" />
-        </inertial>
-        <visual>
-            <origin
-                xyz="0.0 0.05163 0.20994"
-                rpy="0 -1.5708 0" />
-            <geometry>
-                <mesh filename="package://robot_description/meshes/elbow.stl" />
-            </geometry>
-            <material
-                name="">
-                <color
-                rgba="0.79216 0.81961 0.93333 1" />
-            </material>
-        </visual>
-        <collision>
-            <origin
-                xyz="0.0 0.05163 0.20994"
-                rpy="0 -1.5708 0" />
-            <geometry>
-                <mesh filename="package://robot_description/meshes/elbow.stl" />
-            </geometry>
-        </collision>
-    </link>
-    <link
-        name="top_wrist">
-        <inertial>
-            <origin
-                xyz="-9.1053E-08 -0.069257 -1.86629999995759E-07"
-                rpy="0 0 0" />
-            <mass
-                value="0.27721" />
-            <inertia
-                ixx="0.00104290750143942"
-                ixy="4.37155302268076E-09"
-                ixz="-2.45049603914627E-09"
-                iyy="0.000380518373895034"
-                iyz="-7.56009835172156E-09"
-                izz="0.00106006525067445" />
-        </inertial>
-        <visual>
-            <origin
-                xyz="0 0 0.13522"
-                rpy="3.14 0 1.5708" />
-            <geometry>
-                <mesh filename="package://robot_description/meshes/wrist.stl" />
-            </geometry>
-            <material
-                name="">
-                <color
-                rgba="0.79216 0.81961 0.93333 1" />
-            </material>
-        </visual>
-        <collision>
-            <origin
-                xyz="0 0 0.13522"
-                rpy="3.14 0 1.5708" />
-            <geometry>
-                <mesh filename="package://robot_description/meshes/wrist.stl" />
-            </geometry>
-        </collision>
-    </link>
-    <!--############################# Arm Joints #########################################-->
-    <xacro:arm_joint prefix="arm_base" type="continuous" axis="0 0 1" parent="world" child="arm_base" originxyz="0.0 0.0 0.0" originrpy="0 0 0"/>
+    <!--############################# Arm #########################################-->
+    <xacro:arm attach="true"/>
+    <!--############################# Arm Joints ########################################-->
+    <xacro:arm_joint prefix="arm_world" type="fixed" axis="0 0 1" parent="world" child="arm_world" originxyz="0.0 0.0 0.0" originrpy="0 0 0"/>
+    <xacro:arm_joint prefix="arm_base" type="continuous" axis="0 0 1" parent="arm_world" child="arm_base" originxyz="0.0 0.0 0.0" originrpy="0 0 0"/>
     <xacro:arm_joint prefix="shoulder" type="continuous" axis="0 1 0" parent="arm_base" child="bicep" originxyz="-0.05166 0.0 0.20271" originrpy="0 0 1.5708"/>
     <xacro:arm_joint prefix="bottom_wrist" type="continuous" axis="0 1 0" parent="bicep" child="bottom_wrist" originxyz="0.0 -0.05194 0.269" originrpy="0 0 0"/>
     <xacro:arm_joint prefix="elbow" type="continuous" axis="0 0 1" parent="bottom_wrist" child="elbow" originxyz="0.0 0 0.13522" originrpy="0 0 0"/>
     <xacro:arm_joint prefix="top_wrist" type="continuous" axis="0 1 0" parent="elbow" child="top_wrist" originxyz="0.0 0 0.20994" originrpy="0 0 0"/>
-    <!--############################# Arm Transmissions #########################################-->
+    <!--############################# Arm Transmissions ##################################-->
     <xacro:arm_transmission prefix="arm_base"/>
     <xacro:arm_transmission prefix="shoulder"/>
@@ -206,3 +18,6 @@
     <xacro:arm_transmission prefix="elbow"/>
     <xacro:arm_transmission prefix="top_wrist"/>
+    <!--############################# Gazebo ##################################-->
+    <xacro:gazebo_ros_control />
+    <xacro:joint_state_publisher />
 </robot>
