Commit message: launching multiple robots

File: mobile_manipulator_ws/src/robot_description/urdf/gazebo_base_essentials.xacro (robot description, xacro)
@@ -46,3 +46,32 @@
         </gazebo>
     </xacro:macro>
+    <!--############################# Sensors #########################################-->
+    <xacro:macro name="laser_scan">
+        <gazebo reference="laser_link">
+            <sensor type="ray" name="laser">
+            <pose>0 0 0 0 0 0</pose>
+            <visualize>true</visualize>
+            <update_rate>40</update_rate>
+            <ray>
+                <scan>
+                <horizontal>
+                    <samples>720</samples>
+                    <resolution>1</resolution>
+                    <min_angle>-1.570796</min_angle>
+                    <max_angle>1.570796</max_angle>
+                </horizontal>
+                </scan>
+                <range>
+                <min>0.10</min>
+                <max>30.0</max>
+                <resolution>0.01</resolution>
+                </range>
+            </ray>
+            <plugin name="gazebo_ros_head_hokuyo_controller" filename="libgazebo_ros_laser.so">
+                <topicName>/scan</topicName>
+                <frameName>laser_link</frameName>
+            </plugin>
+            </sensor>
+        </gazebo>
+    </xacro:macro>
 </robot>

File: mobile_manipulator_ws/src/robot_description/urdf/mobile_manipulator.urdf.xacro (robot description, xacro)
@@ -62,6 +62,33 @@
   <xacro:wheel_friction prefix="rear_left"/>
   <xacro:wheel_friction prefix="rear_right"/>
+  <!--########################## SENSORS ############################################-->
+  <link name="laser_link">
+    <collision>
+      <origin xyz="0 0 0" rpy="0 0 0"/>
+      <geometry>
+        <box size="0.1 0.1 0.1"/>
+      </geometry>
+    </collision>
+    <visual>
+      <origin xyz="0 0 0" rpy="0 0 0"/>
+      <geometry>
+        <box size="0.05 0.05 0.05"/>
+      </geometry>
+    </visual>
+    <inertial>
+      <mass value="1e-5" />
+      <origin xyz="0 0 0" rpy="0 0 0"/>
+      <inertia ixx="1e-6" ixy="0" ixz="0" iyy="1e-6" iyz="0" izz="1e-6" />
+    </inertial>
+  </link>
+  <joint name="laser_joint" type="fixed">
+    <axis xyz="0 1 0" />
+    <origin xyz="0.350 0 0.115" rpy="0 0 0"/>
+    <parent link="base_link"/>
+    <child link="laser_link"/>
+  </joint>
   <!--############################# GAZEBO #########################################-->
   <xacro:gazebo_ros_control/>
+  <xacro:laser_scan/>
   <xacro:diff_drive_controller/>
   <xacro:joint_state_publisher />
